File: Calender.kicad_pcb (KiCad board)
At the start: 2 copper layers, 94 x 27.5 mm, 51 parts, among them J1 Conn_01x09, J2 USB_C_Receptacle_USB2.0_16P, J3 Power, J4 Screen-2, SW1 RotaryEncoder_Switch, SW2 SW_Push, SW3 SW_Push, SW4 SW_Push, U1 ATSAMD21G18A-A, U3 MCP73871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

Commit message: Fixed the stupid PCB, and added prod files
Parts:
- added D1: SK6812MINI, LED_SMD:LED_SK6812MINI_PLCC4_3.5x3.5mm_P1.75mm, B.Cu at (179.5, 119.0)
- J1: footprint Connector_PinHeader_1.00mm:PinHeader_1x09_P1.00mm_Vertical -> Connector_PinHeader_2.54mm:PinHeader_1x09_P2.54mm_Vertical
- moved SW2 19.6 mm to (223.8, 136.2)
- moved J1 12.1 mm to (235.5, 118.3)
- moved R12 8.09 mm to (226.3, 133.9)
Connections:
- U1 pad 1: unconnected-(U1-PA00-Pad1) -> Net-(D1-DIN)
- U1 pad 33: D+ -> D-
- U1 pad 34: D- -> D+
Routing:
- net GND: track 204.5 -> 160.2 mm, vias 59 -> 67
- net OUT_3.3V: track 173.8 -> 189.0 mm
- net Net-(R12-Pad2): track 17.8 -> 9.52 mm
- net DIN: track 60.0 -> 51.7 mm
- net CS: track 55.3 -> 62.4 mm
- net DC: track 62.6 -> 67.9 mm
- net Net-(D1-DIN): track 0.00 -> 3.53 mm, vias 0 -> 1
- net RST: track 65.3 -> 68.7 mm
- net OUT_5V: track 21.3 -> 23.9 mm
- net BUSY: track 66.9 -> 68.8 mm
- net D+: track 46.6 -> 48.1 mm
- net D-: track 45.8 -> 46.5 mm
- net CLK: track 51.7 -> 52.4 mm, vias 1 -> 2

Commit message: one more time
Parts:
- moved R1 0.33 mm to (152.5, 118.5)
Routing:
- net Net-(J2-CC1): track 2.30 -> 4.73 mm
- net GND: vias 67 -> 68
Changed lines of the file:
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@@
 	(footprint "Resistor_SMD:R_0603_1608Metric"
 		(layer "F.Cu")
-		(at 152.5 118.825 -90)
+		(at 152.5 118.5 -90)
 		(descr "Resistor SMD 0603 (1608 Metric), square (rectangular) end terminal, IPC-7351 nominal, (Body size source: IPC-SM-782 page 72, https://www.pcb-3d.com/wordpress/wp-content/uploads/ipc-sm-782a_amendment_1_and_2.pdf), generated with kicad-footprint-generator")
 		(tags "resistor")
@@
 	)
 	(segment
+		(start 150.37 117.675)
+		(end 150.245 117.8)
+		(width 0.2)
+		(layer "F.Cu")
+		(net 24)
+	)
+	(segment
 		(start 225.9 116.1)
 		(end 225.651 115.851)
@@
 	)
 	(segment
-		(start 152.5 118)
-		(end 150.445 118)
+		(start 152.476626 116.590968)
+		(end 152.5 116.614342)
 		(width 0.2)
 		(layer "F.Cu")
@@
 	)
 	(segment
-		(start 152.5 118)
-		(end 152.5 117)
-		(width 0.2)
-		(layer "F.Cu")
-		(net 24)
-	)
-	(segment
 		(start 185 129.725)
 		(end 185 126.325)
@@
 	)
 	(segment
+		(start 152.5 117.675)
+		(end 150.37 117.675)
+		(width 0.2)
+		(layer "F.Cu")
+		(net 24)
+	)
+	(segment
 		(start 150.245 124.2)
 		(end 152.3 124.2)
@@
 	)
 	(segment
+		(start 152.5 116.614342)
+		(end 152.5 117.675)
+		(width 0.2)
+		(layer "F.Cu")
+		(net 24)
+	)
+	(segment
 		(start 225.651 115.851)
 		(end 220.5 115.851)
@@
 	)
 	(segment
-		(start 150.445 118)
-		(end 150.245 117.8)
-		(width 0.2)
-		(layer "F.Cu")
-		(net 24)
-	)
-	(segment
 		(start 190.5875 119.9125)
 		(end 190.725 120.05)
@@
 	)
 	(via
-		(at 152.5 117)
+		(at 152.476626 116.590968)
 		(size 0.6)
 		(drill 0.3)
@@
 	)
 	(via
+		(at 174.5 120.5)
+		(size 0.6)
+		(drill 0.3)
+		(layers "F.Cu" "B.Cu")
+		(free yes)
+		(net 24)
+	)
+	(via
 		(at 175 124.5)
 		(size 0.6)
@@
 	)
 	(segment
-		(start 151.910936 120.25)
-		(end 150.245 120.25)
+		(start 153.75 120.25)
+		(end 154 120)
 		(width 0.2)
 		(layer "F.Cu")
@@
 	)
 	(segment
-		(start 154 120)
-		(end 153.649 120.351)
-		(width 0.2)
-		(layer "F.Cu")
-		(net 27)
-	)
-	(segment
 		(start 150.245 121.25)
 		(end 149.561176 121.25)
@@
 	)
 	(segment
-		(start 152.011936 120.351)
-		(end 151.910936 120.25)
-		(width 0.2)
-		(layer "F.Cu")
-		(net 27)
-	)
-	(segment
 		(start 187.5 121.0125)
 		(end 187.6 120.9125)
@@
 	)
 	(segment
-		(start 153.649 120.351)
-		(end 152.011936 120.351)
+		(start 149.561176 120.25)
+		(end 150.245 120.25)
 		(width 0.2)
 		(layer "F.Cu")
@@
 	)
 	(segment
-		(start 149.561176 120.25)
-		(end 150.245 120.25)
+		(start 187.6 120.9125)
+		(end 189.4125 120.9125)
 		(width 0.2)
 		(layer "F.Cu")
@@
 	)
 	(segment
-		(start 187.6 120.9125)
-		(end 189.4125 120.9125)
+		(start 150.245 120.25)
+		(end 153.75 120.25)
 		(width 0.2)
 		(layer "F.Cu")
@@
 	)
 	(segment
-		(start 151.196 121.017176)
-		(end 151.196 121.482824)
+		(start 171.101072 117)
+		(end 170.825 117)
 		(width 0.2)
 		(layer "F.Cu")
@@
 	)
 	(segment
-		(start 151.196 121.482824)
-		(end 150.928824 121.75)
+		(start 151.196 121.017176)
+		(end 151.196 121.482824)
 		(width 0.2)
 		(layer "F.Cu")
@@
 	)
 	(segment
-		(start 171.243176 116.581824)
-		(end 170.825 117)
+		(start 151.196 121.482824)
+		(end 150.928824 121.75)
 		(width 0.2)
 		(layer "F.Cu")
@@
 	)
 	(segment
-		(start 171.519248 116.581824)
-		(end 171.243176 116.581824)
+		(start 150.928824 120.75)
+		(end 151.196 121.017176)
 		(width 0.2)
 		(layer "F.Cu")
@@
 	)
 	(segment
-		(start 150.928824 120.75)
-		(end 151.196 121.017176)
+		(start 171.519248 116.581824)
+		(end 171.101072 117)
 		(width 0.2)
 		(layer "F.Cu")
@@
 	)
 	(segment
+		(start 152.5 119.325)
+		(end 152.075 119.75)
+		(width 0.2)
+		(layer "F.Cu")
+		(net 31)
+	)
+	(segment
 		(start 152.4 119.75)
 		(end 150.245 119.75)
 		(width 0.2)
+		(layer "F.Cu")
+		(net 31)
+	)
+	(segment
+		(start 152.075 119.75)
+		(end 150.245 119.75)
+		(width 0.2)

Commit message: fixed the esp32
Connections:
- R12 pad 2: Net-(R12-Pad2) -> Net-(U5-IO0)
- SW2 pad 1: Net-(R12-Pad2) -> Net-(U5-IO0)
- U5 pad 8: OUT_3.3V -> Net-(U5-IO0)
Routing:
- net Net-(U5-IO0): track 0.00 -> 29.3 mm
- net Net-(R12-Pad2): track 9.52 -> 0.00 mm
- net OUT_3.3V: track 189.0 -> 187.0 mm
Changed lines of the file:
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@@
 	(net 63 "Net-(U1-VDDCORE)")
 	(net 64 "Net-(U1-GNDANA)")
-	(net 65 "Net-(R12-Pad2)")
+	(net 65 "Net-(U5-IO0)")
 	(net 66 "Net-(U3-~{PG})")
 	(net 67 "PUSH_NEXT_DAY")
@@
 			(layers "F.Cu" "F.Mask" "F.Paste")
 			(roundrect_rratio 0.25)
-			(net 65 "Net-(R12-Pad2)")
+			(net 65 "Net-(U5-IO0)")
 			(pintype "passive")
 		)
@@
 			(layers "*.Cu" "*.Mask")
 			(remove_unused_layers no)
-			(net 65 "Net-(R12-Pad2)")
+			(net 65 "Net-(U5-IO0)")
 			(pinfunction "1")
 			(pintype "passive")
@@
 			(layers "*.Cu" "*.Mask")
 			(remove_unused_layers no)
-			(net 65 "Net-(R12-Pad2)")
+			(net 65 "Net-(U5-IO0)")
 			(pinfunction "1")
 			(pintype "passive")
@@
 			(size 1.5 0.9)
 			(layers "F.Cu" "F.Mask" "F.Paste")
-			(net 36 "OUT_3.3V")
+			(net 65 "Net-(U5-IO0)")
 			(pinfunction "IO0")
 			(pintype "bidirectional")
@@
 	)
 	(via
-		(at 224.25 133.5)
+		(at 219 132.5)
 		(size 0.6)
 		(drill 0.3)
@@
 	)
 	(segment
-		(start 171.101072 117)
-		(end 170.825 117)
+		(start 151.196 121.017176)
+		(end 151.196 121.482824)
 		(width 0.2)
 		(layer "F.Cu")
@@
 	)
 	(segment
-		(start 151.196 121.017176)
-		(end 151.196 121.482824)
+		(start 171.552864 116.548208)
+		(end 171.101072 117)
 		(width 0.2)
 		(layer "F.Cu")
@@
 	)
 	(segment
-		(start 150.928824 120.75)
-		(end 151.196 121.017176)
+		(start 171.101072 117)
+		(end 170.825 117)
 		(width 0.2)
 		(layer "F.Cu")
@@
 	)
 	(segment
-		(start 171.519248 116.581824)
-		(end 171.101072 117)
+		(start 171.552864 116.466698)
+		(end 171.552864 116.548208)
+		(width 0.2)
+		(layer "F.Cu")
+		(net 30)
+	)
+	(segment
+		(start 150.928824 120.75)
+		(end 151.196 121.017176)
 		(width 0.2)
 		(layer "F.Cu")
@@
 	)
 	(via
-		(at 171.519248 116.581824)
+		(at 171.552864 116.466698)
 		(size 0.6)
 		(drill 0.3)
@@
 	)
 	(segment
+		(start 172 116.101072)
+		(end 172 116.002)
+		(width 0.2)
+		(layer "B.Cu")
+		(net 30)
+	)
+	(segment
 		(start 182.264165 116.002)
 		(end 172 116.002)
@@
 	)
 	(segment
+		(start 171.552864 116.466698)
+		(end 171.634374 116.466698)
+		(width 0.2)
+		(layer "B.Cu")
+		(net 30)
+	)
+	(segment
 		(start 172 116.002)
 		(end 159.498 116.002)
@@
 	)
 	(segment
-		(start 172 116.101072)
-		(end 171.519248 116.581824)
-		(width 0.2)
-		(layer "B.Cu")
-		(net 30)
-	)
-	(segment
-		(start 172 116.002)
+		(start 171.634374 116.466698)
 		(end 172 116.101072)
 		(width 0.2)
@@
 	)
 	(segment
+		(start 208.75 116.1)
+		(end 209.05 116.1)
+		(width 0.4)
+		(layer "F.Cu")
+		(net 36)
+	)
+	(segment
 		(start 224.758636 131.5)
 		(end 224.663308 131.5)
@@
 	)
 	(segment
+		(start 215.374 122.424)
+		(end 215.374 132.029484)
+		(width 0.4)
+		(layer "F.Cu")
+		(net 36)
+	)
+	(segment
 		(start 192 120.667438)
 		(end 192 124.275)
@@
 	)
 	(segment
+		(start 215.720516 132.376)
+		(end 216.949 132.376)
+		(width 0.4)
+		(layer "F.Cu")
+		(net 36)
+	)
+	(segment
 		(start 192.017438 120.65)
 		(end 192 120.667438)
@@
 	)
 	(segment
-		(start 210.111803 117.159803)
-		(end 210.111803 125.538197)
-		(width 0.4)
-		(layer "F.Cu")
-		(net 36)
-	)
-	(segment
 		(start 187 130.5)
 		(end 188.225 130.5)
@@
 	)
 	(segment
-		(start 216.575 132.75)
-		(end 217.825 131.5)
-		(width 0.4)
-		(layer "F.Cu")
-		(net 36)
-	)
-	(segment
-		(start 208.75 126.6)
-		(end 209.05 126.6)
-		(width 0.4)
-		(layer "F.Cu")
-		(net 36)
-	)
-	(segment
 		(start 193 129.775)
 		(end 193 125.275)
@@
 	)
 	(segment
+		(start 216.949 132.376)
+		(end 217.825 131.5)
+		(width 0.4)
+		(layer "F.Cu")
+		(net 36)
+	)
+	(segment
 		(start 198.5 117.175)
 		(end 204 117.175)
@@
 	)
 	(segment
-		(start 209.05 126.6)
-		(end 215.2 132.75)
-		(width 0.4)
-		(layer "F.Cu")
-		(net 36)
-	)
-	(segment
-		(start 209.052 116.1)
-		(end 210.111803 117.159803)
-		(width 0.4)
-		(layer "F.Cu")
-		(net 36)
-	)
-	(segment
 		(start 168.675 116.5)
 		(end 169.175 117)
@@
 	)
 	(segment
-		(start 215.2 132.75)
-		(end 216.575 132.75)
+		(start 209.05 116.1)
+		(end 215.374 122.424)
 		(width 0.4)
 		(layer "F.Cu")
@@
 	)
 	(segment
-		(start 210.111803 125.538197)
-		(end 209.05 126.6)
-		(width 0.4)
-		(layer "F.Cu")
-		(net 36)
-	)
-	(segment
-		(start 208.75 116.1)
-		(end 209.052 116.1)
+		(start 215.374 132.029484)
+		(end 215.720516 132.376)
 		(width 0.4)
 		(layer "F.Cu")
@@
 	)
 	(segment
-		(start 191.751057 118.689122)
-		(end 196.660821 118.689122)
-		(width 0.2)
-		(layer "B.Cu")
-		(net 46)
-	)
-	(segment
 		(start 190.540131 121.326232)
 		(end 191.217535 120.648828)
@@
 	)
 	(segment
-		(start 198.349943 117)
-		(end 218.501057 117)
-		(width 0.2)
-		(layer "B.Cu")
-		(net 46)
-	)
-	(segment
-		(start 228.6945 116.5745)
-		(end 227.1745 116.5745)
+		(start 191.217535 120.648828)
+		(end 191.217535 119.222644)
 		(width 0.2)
 		(layer "B.Cu")
@@
 	)
 	(segment
-		(start 235.5 123.38)
-		(end 228.6945 116.5745)
+		(start 191.217535 119.222644)
+		(end 191.751057 118.689122)
 		(width 0.2)
 		(layer "B.Cu")
@@
 	)
 	(segment
-		(start 218.501057 117)
-		(end 218.926557 116.5745)
+		(start 199.349943 116)
+		(end 228.12 116)
 		(width 0.2)
 		(layer "B.Cu")
@@
 	)
 	(segment
-		(start 218.926557 116.5745)
-		(end 227.1745 116.5745)
+		(start 228.12 116)
+		(end 235.5 123.38)
 		(width 0.2)
 		(layer "B.Cu")
@@
 	)
 	(segment
-		(start 191.217535 119.222644)
-		(end 191.751057 118.689122)
+		(start 191.751057 118.689122)
+		(end 196.660821 118.689122)
 		(width 0.2)
 		(layer "B.Cu")
@@
 	(segment
 		(start 196.660821 118.689122)
-		(end 198.349943 117)
-		(width 0.2)
-		(layer "B.Cu")
-		(net 46)
-	)
-	(segment
-		(start 191.217535 120.648828)
-		(end 191.217535 119.222644)
+		(end 199.349943 116)
 		(width 0.2)
 		(layer "B.Cu")
@@
 		(width 0.2)
 		(layer "F.Cu")
+		(net 65)
+	)
+	(segment
+		(start 208.75 126.6)
+		(end 209.1 126.6)
+		(width 0.2)
+		(layer "F.Cu")
+		(net 65)
+	)
+	(segment
+		(start 209.1 126.6)
+		(end 216.436567 133.936567)
+		(width 0.2)
+		(layer "F.Cu")
+		(net 65)
+	)
+	(segment
+		(start 216.436567 133.936567)
+		(end 225.449875 133.936567)
+		(width 0.2)
+		(layer "F.Cu")
