File: Calender.kicad_sch (KiCad schematic)
At the start: 52 parts, among them J1 Conn_01x09, J2 USB_C_Receptacle_USB2.0_16P, J3 Power, J4 Screen-2, SW1 RotaryEncoder_Switch, SW2 SW_Push, SW3 SW_Push, SW4 SW_Push, U1 ATSAMD21G18A-A, U3 MCP73871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

Commit message: Fixed the stupid PCB, and added prod files
Parts:
- removed TP6, TP7: TestPoint, Connector_Pin:Pin_D1.0mm_L10.0mm_LooseFit, symbol Connector:TestPoint
- added D1: SK6812MINI, LED_SMD:LED_SK6812MINI_PLCC4_3.5x3.5mm_P1.75mm, symbol LED:SK6812MINI
Connections:
- net D+: now also U1.34 (PA25); no longer U1.33 (PA24)
- net D-: now also U1.33 (PA24); no longer U1.34 (PA25)
- net GND: now also D1.2 (VSS)
- net OUT_5V: now also D1.4 (VDD)
- net at U1.1 (PA00): now also D1.3 (DIN)
- no-connect marks 26 -> 25
Other:
- moved on the sheet: R15

Commit message: fixed the esp32
Connections:
- net OUT_3.3V: no longer U5.8 (IO0)
- net at R12.2, SW2.1: now also U5.8 (IO0)
Other:
- moved on the sheet: R12, SW2
Changed lines of the file:
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@@
 	)
 	(junction
-		(at 261.62 123.19)
-		(diameter 0)
-		(color 0 0 0 0)
-	)
-	(junction
 		(at 177.8 91.44)
 		(diameter 0)
@@
 		(color 0 0 0 0)
 	)
+	(junction
+		(at 261.62 123.19)
+		(diameter 0)
+		(color 0 0 0 0)
+	)
 	(no_connect
 		(at 257.81 138.43)
@@
 	(wire
 		(pts
+			(xy 261.62 115.57) (xy 261.62 114.3)
+		)
+		(stroke
+			(width 0)
+			(type default)
+		)
+	)
+	(wire
+		(pts
 			(xy 40.64 116.84) (xy 41.91 116.84)
 		)
@@
 	(wire
 		(pts
-			(xy 261.62 123.19) (xy 261.62 121.92)
-		)
-		(stroke
-			(width 0)
-			(type default)
-		)
-	)
-	(wire
-		(pts
 			(xy 186.69 111.76) (xy 196.85 111.76)
 		)
@@
 	(global_label "OUT_3.3V"
 		(shape input)
-		(at 261.62 121.92 90)
+		(at 261.62 114.3 90)
 		(fields_autoplaced yes)
 		(effects
@@
 		)
 		(property "Intersheetrefs" "${INTERSHEET_REFS}"
-			(at 261.62 110.2262 90)
+			(at 261.62 102.6062 90)
 			(effects
 				(font
@@
 	(symbol
 		(lib_id "power:GND")
-		(at 261.62 140.97 90)
+		(at 271.78 123.19 0)
 		(unit 1)
 		(exclude_from_sim no)
@@
 		(fields_autoplaced yes)
 		(property "Reference" "#PWR029"
-			(at 267.97 140.97 0)
+			(at 271.78 129.54 0)
 			(effects
 				(font
@@
 		)
 		(property "Value" "GND"
-			(at 265.43 140.9699 90)
+			(at 271.78 128.27 0)
 			(effects
 				(font
 					(size 1.27 1.27)
 				)
-				(justify right)
 			)
 		)
 		(property "Footprint" ""
-			(at 261.62 140.97 0)
+			(at 271.78 123.19 0)
 			(effects
 				(font
@@
 		)
 		(property "Datasheet" ""
-			(at 261.62 140.97 0)
+			(at 271.78 123.19 0)
 			(effects
 				(font
@@
 		)
 		(property "Description" "Power symbol creates a global label with name \"GND\" , ground"
-			(at 261.62 140.97 0)
+			(at 271.78 123.19 0)
 			(effects
 				(font
@@
 	(symbol
 		(lib_id "Device:R")
-		(at 261.62 127 0)
+		(at 261.62 119.38 0)
 		(unit 1)
 		(exclude_from_sim no)
@@
 		(dnp no)
 		(property "Reference" "R12"
-			(at 263.906 126.746 90)
+			(at 258.826 119.38 90)
 			(effects
 				(font
@@
 		)
 		(property "Value" "10k"
-			(at 261.62 127 90)
+			(at 261.62 119.38 90)
 			(effects
 				(font
@@
 		)
 		(property "Footprint" "Resistor_SMD:R_0603_1608Metric"
-			(at 259.842 127 90)
+			(at 259.842 119.38 90)
 			(effects
 				(font
@@
 		)
 		(property "Datasheet" "~"
-			(at 261.62 127 0)
+			(at 261.62 119.38 0)
 			(effects
 				(font
@@
 		)
 		(property "Description" "Resistor"
-			(at 261.62 127 0)
+			(at 261.62 119.38 0)
 			(effects
 				(font
@@
 	(symbol
 		(lib_id "Switch:SW_Push")
-		(at 261.62 135.89 270)
+		(at 266.7 123.19 0)
 		(unit 1)
 		(exclude_from_sim no)
@@
 		(on_board yes)
 		(dnp no)
-		(fields_autoplaced yes)
 		(property "Reference" "SW2"
-			(at 265.43 134.6199 90)
+			(at 267.462 116.078 0)
 			(effects
 				(font
 					(size 1.27 1.27)
 				)
-				(justify left)
 			)
 		)
 		(property "Value" "SW_Push"
-			(at 265.43 137.1599 90)
+			(at 267.462 118.618 0)
 			(effects
 				(font
 					(size 1.27 1.27)
 				)
-				(justify left)
 			)
 		)
 		(property "Footprint" "Button_Switch_THT:SW_PUSH_6mm"
-			(at 266.7 135.89 0)
+			(at 266.7 118.11 0)
 			(effects
 				(font
@@
 		)
 		(property "Datasheet" "~"
-			(at 266.7 135.89 0)
+			(at 266.7 118.11 0)
 			(effects
 				(font
@@
 		)
 		(property "Description" "Push button switch, generic, two pins"
-			(at 261.62 135.89 0)
+			(at 266.7 123.19 0)
 			(effects
 				(font
@@
 		(on_board yes)
 		(dnp no)
-		(fields_autoplaced yes)
 		(property "Reference" "U5"
-			(at 247.2533 115.57 0)
+			(at 247.65 105.664 0)
 			(effects
 				(font
@@
 		)
 		(property "Value" "ESP-WROOM-02"
-			(at 247.2533 118.11 0)
+			(at 239.268 103.124 0)
 			(effects
 				(font
